Commit message: map: no-go zone editing+overlay, persistent maps, custom planner safety
Implements editable maps with no-go zones and makes mapping persistence the
default for stability:

- occupancy.py: new forbidden (no-go) mask kept separate from log-odds so a
  lidar beam through a zone can't un-forbid it; brush/erase/clear editing,
  strokes over world-space lines, folded into the planner's blocked mask
  (radius-inflated, immune to allow_unknown), and persisted in the map.
- nav_node.py: polls a /dev/shm edit-request file (token-idempotent, no file
  race), applies strokes/clear, rewrites the map + no-go blob, and persists
  edits immediately; map_server path now expanduser + mkdir'd.
- index.html: Map view gains a Goal / No-go / No-go-erase / Clear-zones
  toolbar + brush slider; forbidden zones render as an amber overlay;
  stroke paint posts on pointer-up (one request per stroke).
- web_server.py: GET /map/nogo (serve overlay blob) + POST /map/nogo/stroke
  and /map/nogo/clear (atomic handoff to slam_nav).
- robot.yaml: enable map_store + autosave_period by default so the grid
  (and no-go zones) persists across boot.
- OpenRouter key loading from memory/openrouter_key into bringup/sim/visualize
  and stack.sh; deploy.sh also pushes llm.json; cognition reports model_for().

File: src/robot_bringup/urdf/nano.urdf.xacro (robot description, xacro)
@@ -16,5 +16,4 @@
 -->
 <robot name="nano" xmlns:xacro="http://www.ros.org/wiki/xacro">
-  <xacro:property name="pi" value="3.14159265359"/>
   <xacro:property name="wheel_radius" value="0.0335"/>
   <xacro:property name="wheel_separation" value="0.16"/>
